File: board/m8/m8.kicad_pcb (KiCad board)
At the start: 2 copper layers, 50 x 25 mm, 11 parts, among them J1 program, SW1 B3F-4000, U1 CH32V003f4p6

Commit message: rev2 with sugestions from Chip
Parts:
- removed C2: 100n, Capacitor_SMD:C_0805_2012Metric_Pad1.18x1.45mm_HandSolder
- C1: value 10u -> 100n
- moved C1 12.6 mm to (159.8, 111.0)
- moved SW1 9.47 mm to (129.9, 106.2), turned to -90 degrees
Connections:
- SW1 pad 1: unconnected-(SW1-Pad1) -> GND
- SW1 pad 2: GND -> Net-(U1-PC0_T2CH3)
- SW1 pad 3: Net-(U1-PC0_T2CH3) -> unconnected-(SW1-Pad3)
Routing:
- net Net-(U1-PC0_T2CH3): track 59.4 -> 46.9 mm
- net GND: track 65.9 -> 56.6 mm, vias 3 -> 2
- net VCC: track 132.2 -> 125.9 mm

Commit message: fixed bugs!
Connections:
- SW1 pad 1: GND -> unconnected-(SW1-Pad1)
- SW1 pad 3: unconnected-(SW1-Pad3) -> GND
Routing:
- net GND: track 56.6 -> 64.6 mm
Changed lines of the file:
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@@
 	(net 22 "Net-(J1-Pin_6)")
 	(net 23 "Net-(J1-Pin_4)")
-	(net 24 "unconnected-(SW1-Pad3)")
+	(net 24 "unconnected-(SW1-Pad1)")
 	(net 25 "unconnected-(SW1-Pad4)")
 	(footprint "Package_SO:TSSOP-20_4.4x6.5mm_P0.65mm"
@@
 			(layers "*.Cu" "*.Mask")
 			(remove_unused_layers no)
-			(net 8 "GND")
+			(net 24 "unconnected-(SW1-Pad1)")
 			(pinfunction "1")
 			(pintype "unspecified")
@@
 			(layers "*.Cu" "*.Mask")
 			(remove_unused_layers no)
-			(net 24 "unconnected-(SW1-Pad3)")
+			(net 8 "GND")
 			(pinfunction "3")
 			(pintype "unspecified")
@@
 	)
 	(segment
+		(start 160.2 110.35)
+		(end 159.8 109.95)
+		(width 0.4)
+		(layer "F.Cu")
+		(net 8)
+	)
+	(segment
 		(start 146.5 112.4)
 		(end 145.1 112.4)
@@
 	(segment
 		(start 159.299999 109.006218)
-		(end 159.299999 110.35)
+		(end 159.299999 109.449999)
 		(width 0.4)
 		(layer "F.Cu")
@@
 	)
 	(segment
-		(start 146.5 114.9)
-		(end 146.5 112.4)
+		(start 161.9375 110.35)
+		(end 160.2 110.35)
 		(width 0.4)
 		(layer "F.Cu")
@@
 	)
 	(segment
-		(start 161.9375 110.35)
-		(end 160.2 110.35)
+		(start 146.5 114.9)
+		(end 146.5 112.4)
 		(width 0.4)
 		(layer "F.Cu")
@@
 	)
 	(segment
-		(start 160.2 110.35)
+		(start 159.299999 109.449999)
 		(end 159.8 109.95)
 		(width 0.4)
@@
 	)
 	(segment
-		(start 158.553616 115.75)
-		(end 158.578616 115.725)
-		(width 0.2)
+		(start 138 105.803616)
+		(end 138 111.4)
+		(width 0.4)
 		(layer "B.Cu")
 		(net 8)
 	)
 	(segment
-		(start 145.1 112.4)
-		(end 158.578616 112.4)
+		(start 140.803616 103)
+		(end 138 105.803616)
+		(width 0.4)
+		(layer "B.Cu")
+		(net 8)
+	)
+	(segment
+		(start 138 111.4)
+		(end 139 112.4)
 		(width 0.4)
 		(layer "B.Cu")
@@
 	)
 	(segment
-		(start 138 112.4)
-		(end 136.1 112.4)
+		(start 158.578616 112.078616)
+		(end 159.1 112.6)
+		(width 0.4)
+		(layer "B.Cu")
+		(net 8)
+	)
+	(segment
+		(start 145.1 112.4)
+		(end 158.578616 112.4)
 		(width 0.4)
 		(layer "B.Cu")
@@
 	)
 	(segment
-		(start 138 105.803616)
-		(end 138 112.4)
+		(start 158.603616 112.425)
+		(end 158.578616 112.4)
 		(width 0.4)
 		(layer "B.Cu")
@@
 	)
 	(segment
-		(start 141 112.4)
-		(end 138 112.4)
+		(start 125.75 109.3)
+		(end 124.95 108.5)
 		(width 0.4)
 		(layer "B.Cu")
@@
 	)
 	(segment
-		(start 136.1 112.4)
-		(end 129.95 106.25)
+		(start 145.1 112.4)
+		(end 141 112.4)
 		(width 0.4)
 		(layer "B.Cu")
@@
 	)
 	(segment
-		(start 140.803616 103)
-		(end 138 105.803616)
+		(start 158.578616 109.727601)
+		(end 158.578616 112.078616)
 		(width 0.4)
 		(layer "B.Cu")
@@
 	)
 	(segment
-		(start 145.1 112.4)
+		(start 158.925 112.425)
+		(end 158.603616 112.425)
+		(width 0.4)
+		(layer "B.Cu")
+		(net 8)
+	)
+	(segment
+		(start 137.95 109.3)
+		(end 125.75 109.3)
+		(width 0.4)
+		(layer "B.Cu")
+		(net 8)
+	)
+	(segment
+		(start 139 112.4)
 		(end 141 112.4)
 		(width 0.4)
@@
 	)
 	(segment
+		(start 159.1 112.6)
+		(end 158.925 112.425)
+		(width 0.4)
+		(layer "B.Cu")
+		(net 8)
+	)
+	(segment
+		(start 124.95 108.5)
+		(end 124.95 106.25)
+		(width 0.4)
+		(layer "B.Cu")
+		(net 8)
+	)
+	(segment
+		(start 138 109.25)
+		(end 137.95 109.3)
+		(width 0.4)
+		(layer "B.Cu")
+		(net 8)
+	)
+	(segment
 		(start 159.299999 109.006218)
 		(end 158.578616 109.727601)
@@
 		(start 160.175 111.65)
 		(end 159.8 112.025)
-		(width 0.2)
+		(width 0.4)
 		(layer "F.Cu")
 		(net 17)
