File: board/m8/m8.kicad_sch (KiCad schematic)
At the start: 11 parts, among them J1 program, SW1 B3F-4000, U1 CH32V003f4p6

Commit message: Found bugs fixed them!
Parts:
- LED1: footprint LED_SMD:LED_ROHM_SMLVN6 -> LED_SMD:LED_RGB_5050-6
- LS1: footprint Buzzer_Beeper:Buzzer_12x9.5RM7.6 -> Library:Buzzer_12x8.4RM6.6
Changed lines of the file:
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@@
 			)
 		)
-		(property "Footprint" "LED_SMD:LED_ROHM_SMLVN6"
+		(property "Footprint" "LED_SMD:LED_RGB_5050-6"
 			(at 128.27 71.12 0)
 			(effects
@@
 			)
 		)
-		(property "Footprint" "Buzzer_Beeper:Buzzer_12x9.5RM7.6"
+		(property "Footprint" "Library:Buzzer_12x8.4RM6.6"
 			(at 123.571 31.75 0)
 			(effects

Commit message: rev2 with sugestions from Chip
Parts:
- removed C2: 100n, Capacitor_SMD:C_0805_2012Metric_Pad1.18x1.45mm_HandSolder, symbol Device:C
- C1: value 10u -> 100n
Connections:
- net GND: now also SW1.1; no longer SW1.2
- net at U1.10 (PC0_T2CH3): now also SW1.2; no longer SW1.3
Other:
- moved on the sheet: SW1
Changed lines of the file:
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@@
-	)
-	(junction
-		(at 52.07 91.44)
-		(diameter 0)
-		(color 0 0 0 0)
-	)
-	(junction
-		(at 52.07 69.85)
-		(diameter 0)
-		(color 0 0 0 0)
 	)
 	(junction
@@
 	(wire
 		(pts
-			(xy 116.84 62.23) (xy 120.65 62.23)
-		)
-		(stroke
-			(width 0)
-			(type default)
-		)
-	)
-	(wire
-		(pts
 			(xy 107.95 74.93) (xy 116.84 74.93)
 		)
@@
 	(wire
 		(pts
-			(xy 116.84 62.23) (xy 116.84 74.93)
-		)
-		(stroke
-			(width 0)
-			(type default)
-		)
-	)
-	(wire
-		(pts
-			(xy 44.45 91.44) (xy 52.07 91.44)
+			(xy 44.45 91.44) (xy 64.77 91.44)
 		)
 		(stroke
@@
 	(wire
 		(pts
+			(xy 116.84 59.69) (xy 121.92 59.69)
+		)
+		(stroke
+			(width 0)
+			(type default)
+		)
+	)
+	(wire
+		(pts
 			(xy 113.03 105.41) (xy 113.03 59.69)
 		)
@@
 	(wire
 		(pts
-			(xy 52.07 91.44) (xy 64.77 91.44)
-		)
-		(stroke
-			(width 0)
-			(type default)
-		)
-	)
-	(wire
-		(pts
 			(xy 144.78 80.01) (xy 149.86 80.01)
 		)
@@
 	(wire
 		(pts
-			(xy 161.29 59.69) (xy 166.37 59.69)
-		)
-		(stroke
-			(width 0)
-			(type default)
-		)
-	)
-	(wire
-		(pts
 			(xy 113.03 59.69) (xy 107.95 59.69)
 		)
@@
 	(wire
 		(pts
-			(xy 52.07 76.2) (xy 52.07 69.85)
-		)
-		(stroke
-			(width 0)
-			(type default)
-		)
-	)
-	(wire
-		(pts
 			(xy 133.35 80.01) (xy 137.16 80.01)
 		)
@@
 	(wire
 		(pts
-			(xy 52.07 69.85) (xy 64.77 69.85)
-		)
-		(stroke
-			(width 0)
-			(type default)
-		)
-	)
-	(wire
-		(pts
 			(xy 71.12 69.85) (xy 71.12 57.15)
 		)
@@
 	(wire
 		(pts
+			(xy 162.56 59.69) (xy 166.37 59.69)
+		)
+		(stroke
+			(width 0)
+			(type default)
+		)
+	)
+	(wire
+		(pts
 			(xy 44.45 83.82) (xy 44.45 91.44)
 		)
@@
 	(wire
 		(pts
-			(xy 44.45 69.85) (xy 52.07 69.85)
-		)
-		(stroke
-			(width 0)
-			(type default)
-		)
-	)
-	(wire
-		(pts
-			(xy 52.07 83.82) (xy 52.07 91.44)
+			(xy 44.45 69.85) (xy 64.77 69.85)
 		)
 		(stroke
@@
 		(pts
 			(xy 107.95 97.79) (xy 118.11 97.79)
+		)
+		(stroke
+			(width 0)
+			(type default)
+		)
+	)
+	(wire
+		(pts
+			(xy 116.84 59.69) (xy 116.84 74.93)
 		)
 		(stroke
@@
 	(symbol
 		(lib_id "2024-05-26_01-20-13:B3F-4000")
-		(at 120.65 59.69 0)
-		(unit 1)
-		(exclude_from_sim no)
-		(in_bom yes)
-		(on_board yes)
-		(dnp no)
-		(fields_autoplaced yes)
+		(at 162.56 59.69 0)
+		(mirror y)
+		(unit 1)
+		(exclude_from_sim no)
+		(in_bom yes)
+		(on_board yes)
+		(dnp no)
 		(property "Reference" "SW1"
-			(at 140.97 49.53 0)
+			(at 142.24 49.53 0)
 			(effects
 				(font
@@
 		)
 		(property "Value" "B3F-4000"
-			(at 140.97 52.07 0)
+			(at 142.24 52.07 0)
 			(effects
 				(font
@@
 		)
 		(property "Footprint" "SW_B3F-4000_OMR"
-			(at 120.65 59.69 0)
+			(at 162.56 59.69 0)
 			(effects
 				(font
@@
 		)
 		(property "Datasheet" "B3F-4000"
-			(at 120.65 59.69 0)
+			(at 162.56 59.69 0)
 			(effects
 				(font
@@
 		)
 		(property "Description" ""
-			(at 120.65 59.69 0)
+			(at 162.56 59.69 0)
 			(effects
 				(font
@@
 				(path "/a6d87edb-2eb8-4205-ac8c-5ddfea66c6c8"
 					(reference "R1")
-					(unit 1)
-				)
-			)
-		)
-	)
-	(symbol
-		(lib_id "Device:C")
-		(at 52.07 80.01 0)
-		(unit 1)
-		(exclude_from_sim no)
-		(in_bom yes)
-		(on_board yes)
-		(dnp no)
-		(fields_autoplaced yes)
-		(property "Reference" "C2"
-			(at 55.88 78.7399 0)
-			(effects
-				(font
-					(size 1.27 1.27)
-				)
-				(justify left)
-			)
-		)
-		(property "Value" "100n"
-			(at 55.88 81.2799 0)
-			(effects
-				(font
-					(size 1.27 1.27)
-				)
-				(justify left)
-			)
-		)
-		(property "Footprint" "Capacitor_SMD:C_0805_2012Metric_Pad1.18x1.45mm_HandSolder"
-			(at 53.0352 83.82 0)
-			(effects
-				(font
-					(size 1.27 1.27)
-				)
-				(hide yes)
-			)
-		)
-		(property "Datasheet" "~"
-			(at 52.07 80.01 0)
-			(effects
-				(font
-					(size 1.27 1.27)
-				)
-				(hide yes)
-			)
-		)
-		(property "Description" "Unpolarized capacitor"
-			(at 52.07 80.01 0)
-			(effects
-				(font
-					(size 1.27 1.27)
-				)
-				(hide yes)
-			)
-		)
-		(pin "2"
-		)
-		(pin "1"
-		)
-		(instances
-			(project "m8"
-				(path "/a6d87edb-2eb8-4205-ac8c-5ddfea66c6c8"
-					(reference "C2")
 					(unit 1)
 				)
@@
 			)
 		)
-		(property "Value" "10u"
+		(property "Value" "100n"
 			(at 68.58 81.2799 0)
 			(effects

Commit message: fixed bugs!
Connections:
- net GND: now also SW1.3; no longer SW1.1
Changed lines of the file:
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@@
+	(wire
+		(pts
+			(xy 162.56 62.23) (xy 167.64 62.23)
+		)
+		(stroke
+			(width 0)
+			(type default)
+		)
+	)
 	(wire
 		(pts
@@
 		(pts
 			(xy 107.95 80.01) (xy 120.65 80.01)
-		)
-		(stroke
-			(width 0)
-			(type default)
-		)
-	)
-	(wire
-		(pts
-			(xy 162.56 59.69) (xy 166.37 59.69)
 		)
 		(stroke
@@
 	(symbol
 		(lib_id "power:GND")
-		(at 166.37 59.69 90)
+		(at 167.64 62.23 90)
 		(unit 1)
 		(exclude_from_sim no)
@@
 		(fields_autoplaced yes)
 		(property "Reference" "#PWR06"
-			(at 172.72 59.69 0)
+			(at 173.99 62.23 0)
 			(effects
 				(font
@@
 		)
 		(property "Value" "GND"
-			(at 170.18 59.6899 90)
+			(at 171.45 62.2299 90)
 			(effects
 				(font
@@
 		)
 		(property "Footprint" ""
-			(at 166.37 59.69 0)
+			(at 167.64 62.23 0)
 			(effects
 				(font
@@
 		)
 		(property "Datasheet" ""
-			(at 166.37 59.69 0)
+			(at 167.64 62.23 0)
 			(effects
 				(font
@@
 		)
 		(property "Description" "Power symbol creates a global label with name \"GND\" , ground"
-			(at 166.37 59.69 0)
-			(effects
-				(font
+			(at 167.64 62.23 0)
+			(effects
+				(font

Commit message: got fancy anamated lights started
Parts:
- R1, R3: value 10 -> 1
Changed lines of the file:
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@@
 			)
 		)
-		(property "Value" "10"
+		(property "Value" "1"
 			(at 142.494 82.804 90)
 			(effects
@@
 			)
 		)
-		(property "Value" "10"
+		(property "Value" "1"
 			(at 142.494 72.644 90)
 			(effects
